File: 003_KBD_ATmega32u2Test.sch (KiCad schematic (older format))
At the start: 18 parts

Commit message: 回路図の更新(ATMEGA32U4へ変更、OLED追加)
Parts:
- removed U?: ATmega32U2-AU, Package_QFP:TQFP-32_7x7mm_P0.8mm, symbol MCU_Microchip_ATmega:ATmega32U2-AU
- added D1, D2, D3, D4: D, Diode_SMD:D_SOD-123, symbol Device:D
- added J1: Conn_01x04_Male, Connector_PinSocket_2.54mm:PinSocket_1x04_P2.54mm_Vertical, symbol Connector:Conn_01x04_Male
- added SW1, SW2, SW3, SW4: SW_PUSH, KBD_foostan:CherryMX_Hotswap, symbol KBD_foostan:SW_PUSH
- added U1: ATmega32U4-AU, Package_QFP:TQFP-44_10x10mm_P0.8mm, symbol MCU_Microchip_ATmega:ATmega32U4-AU
- C1, C2, C3, C4, C5, C6: renamed from C?; footprint (none) -> Capacitor_Tantalum_SMD:CP_EIA-1608-08_AVX-J
- C7, C8: renamed from C?; value 22p -> 9p; footprint (none) -> Capacitor_Tantalum_SMD:CP_EIA-1608-08_AVX-J
- J2: renamed from J?; footprint (none) -> Connector_USB:USB_C_Receptacle_HRO_TYPE-C-31-M-12
- R1, R2, R5, R6: renamed from R?; footprint (none) -> Resistor_SMD:R_0603_1608Metric
- R3, R4: renamed from R?; value 22 -> 5.1k; footprint (none) -> Resistor_SMD:R_0603_1608Metric
- RST1: renamed from RST?; footprint (none) -> KBD_foostan:ResetSW_1side
- Y1: renamed from Y?; footprint (none) -> Crystal:Crystal_SMD_3225-4Pin_3.2x2.5mm
Connections:
- net GND: now also J1.1 (Pin_1), U1.15 (GND), U1.23 (GND), U1.35 (GND), U1.43 (GND), U1.5 (UGND)
- net VCC: now also J1.2 (Pin_2), U1.14 (VCC), U1.2 (UVCC), U1.24 (AVCC), U1.34 (VCC), U1.44 (AVCC), U1.7 (VBUS)
- net d+: now also U1.4 (D+)
- net d-: now also U1.3 (D-)
- net reset: now also U1.13 (~RESET)
- net xtal1: now also U1.17 (XTAL1)
- net xtal2: now also U1.16 (XTAL2)
- net at R1.2: now also U1.33 (~HWB~/PE2)
- net at C1.2: now also U1.6 (UCAP)
- new net: D1.2 (A), SW1.1
- new net: D2.2 (A), SW2.1
- new net: D4.2 (A), SW4.1
- new net: D3.2 (A), SW3.1
- new net SCL: J1.3 (Pin_3), U1.18 (PD0)
- new net SDA: J1.4 (Pin_4), U1.19 (PD1)
- new net col0: SW1.2, SW2.2, U1.29 (PB5)
- new net col1: SW3.2, SW4.2, U1.28 (PB4)
- new net row0: D1.1 (K), D3.1 (K), U1.27 (PD7)
- new net row1: D2.1 (K), D4.1 (K), U1.30 (PB6)
- no-connect marks 2 -> 22
Other:
- moved on the sheet: C1, C2, C3, C4, C5, C6, C7, C8, J2, R1, R2, R3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
